Commit message: chore: repo cleaning

File: workspace/src/robot_description/urdf/ur5_no_ee.urdf (robot description, URDF)
Before this commit: robot ur5_rg2, 7 links, 6 joints
Links:
- link base_link: geometry collision mesh filename=package://robot_description/meshes/collision/ur5/base.stl; visual mesh filename=package://robot_description/meshes/visual/ur5/base.dae
- link forearm_link: geometry collision mesh filename=package://robot_description/meshes/collision/ur5/forearm.stl; visual mesh filename=package://robot_description/meshes/visual/ur5/forearm.dae
- link shoulder_link: geometry collision mesh filename=package://robot_description/meshes/collision/ur5/shoulder.s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; visual mesh filename=package://robot_description/meshes/visual/ur5/shoulder.dae
- link upper_arm_link: geometry collision mesh filename=package://robot_description/meshes/collision/ur5/upperarm.s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; visual mesh filename=package://robot_description/meshes/visual/ur5/upperarm.dae
- link wrist_1_link: geometry collision mesh filename=package://robot_description/meshes/collision/ur5/wrist1.stl; visual mesh filename=package://robot_description/meshes/visual/ur5/wrist1.dae
- link wrist_2_link: geometry collision mesh filename=package://robot_description/meshes/collision/ur5/wrist2.stl; visual mesh filename=package://robot_description/meshes/visual/ur5/wrist2.dae
- link wrist_3_link: geometry collision mesh filename=package://robot_description/meshes/collision/ur5/wrist3.stl; visual mesh filename=package://robot_description/meshes/visual/ur5/wrist3.dae

File: workspace/src/robot_description/urdf/ur5_no_ee_gazebo.urdf (robot description, URDF)
Before this commit: robot ur5_rg2, 7 links, 6 joints
Links:
- link base_link: geometry collision mesh filename=package://meshes/collision/ur5/base.stl; visual mesh filename=package://meshes/visual/ur5/base.dae
- link forearm_link: geometry collision mesh filename=package://meshes/collision/ur5/forearm.stl; visual mesh filename=package://meshes/visual/ur5/forearm.dae
- link shoulder_link: geometry collision mesh filename=package://meshes/collision/ur5/shoulder.stl; visual mesh filename=package://meshes/visual/ur5/shoulder.dae
- link upper_arm_link: geometry collision mesh filename=package://meshes/collision/ur5/upperarm.stl; visual mesh filename=package://meshes/visual/ur5/upperarm.dae
- link wrist_1_link: geometry collision mesh filename=package://meshes/collision/ur5/wrist1.stl; visual mesh filename=package://meshes/visual/ur5/wrist1.dae
- link wrist_2_link: geometry collision mesh filename=package://meshes/collision/ur5/wrist2.stl; visual mesh filename=package://meshes/visual/ur5/wrist2.dae
- link wrist_3_link: geometry collision mesh filename=package://meshes/collision/ur5/wrist3.stl; visual mesh filename=package://meshes/visual/ur5/wrist3.dae
